File: pcb/ir03/ir03.brd (EAGLE design)
At the start: 63.5 x 55.5 mm, 15 parts

Commit message: UPD: pcb
Parts:
- Q2: value (none) -> 2SK4017
Changed lines of the file:
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@@
 <attribute name="VALUE" x="27.305" y="34.671" size="1.27" layer="27" ratio="10" rot="R180"/>
 </element>
-<element name="Q2" library="adafruit" package="TO220V" value="" x="15.24" y="38.1" smashed="yes">
+<element name="Q2" library="adafruit" package="TO220V" value="2SK4017" x="15.24" y="38.1" smashed="yes">
 <attribute name="NAME" x="10.16" y="32.0548" size="1.27" layer="25" ratio="10"/>
 <attribute name="VALUE" x="10.16" y="30.48" size="1.27" layer="27" ratio="10"/>
