File: pcb/ir03/ir03.sch (EAGLE design)
At the start: 15 parts

Commit message: UPD: pcb
Parts:
- Q2: value (none) -> 2SK4017
Changed lines of the file:
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@@
 <part name="LED7" library="adafruit" deviceset="LED" device="3MM"/>
 <part name="LED8" library="adafruit" deviceset="LED" device="3MM"/>
-<part name="Q2" library="adafruit" deviceset="MOSFET-N" device="GDS_TO220V"/>
+<part name="Q2" library="adafruit" deviceset="MOSFET-N" device="GDS_TO220V" value="2SK4017"/>
 <part name="R5" library="rcl" library_urn="urn:adsk.eagle:library:334" deviceset="R-US_" device="0204/5" package3d_urn="urn:adsk.eagle:package:23488/1" value="10Ω"/>
 <part name="R6" library="rcl" library_urn="urn:adsk.eagle:library:334" deviceset="R-US_" device="0204/5" package3d_urn="urn:adsk.eagle:package:23488/1" value="10Ω"/>
